File: WLED_ESP8266_molex_microfit/_autosave-WLED_ESP8266_molex_microfit.kicad_sch (KiCad schematic)
At the start: 62 parts, among them J1 Molex Micro-fit 2x1, J2 Molex Micro-fit 3x1, J3 Molex Micro-fit 2x1, J4 Molex Micro-fit 2x1, J6 Molex Micro-fit 2x1, J7 Molex Micro-fit 3x1, J8 Molex Micro-fit 3x1, Q1 AO3401A, Q2 AO3401A, U1 ESP-12F, U2 TPS54331DDAR, U3 TXS0102DCT, U4 TXS0102DCT, U6 ME6211A33M3G-N

Commit message: V1 completed
Connections:
- net +3.3V is gone; now on net +3V3: JP4.1 (A), TP1.1
- net GPIO_15: now also U1.16 (GPIO15)
- net VIN_F: now also C1.1, C2.1, F1.2, R3.1, U2.2 (VIN)
- net Q1_Drain: now reaches J3.2 (Pin_2), Q1.3 (D)
- net TPS_PH: now reaches C4.2, D1.1 (K), L1.1, U2.8 (PH)
- net Q2_Drain: now reaches J4.2 (Pin_2), Q2.3 (D)
