File: WLED_ESP8266_molex_microfit/WLED_ESP8266_molex_microfit.kicad_sch (KiCad schematic)
At the start: 65 parts, among them J1 Molex Micro-fit 2x1, J2 Molex Micro-fit 3x1, J3 Molex Micro-fit 2x1, J4 Molex Micro-fit 2x1, J5 USB_B_Micro, J6 Molex Micro-fit 2x1, J7 Molex Micro-fit 3x1, J8 Molex Micro-fit 3x1, Q1 AO3401A, Q2 AO3401A, U1 ESP-12F, U2 TPS54331DDAR, U3 TXS0102DCT, U4 TXS0102DCT, U6 ME6211A33M3G-N

Commit message: feedback implemented
Parts:
- removed TP1: +3.3V, TestPoint:TestPoint_Pad_D1.5mm, symbol Connector:TestPoint
- removed TP2: TX, TestPoint:TestPoint_Pad_D1.5mm, symbol Connector:TestPoint
- removed TP3: RX, TestPoint:TestPoint_Pad_D1.5mm, symbol Connector:TestPoint
- removed TP4: GND, TestPoint:TestPoint_Pad_D1.5mm, symbol Connector:TestPoint
- added J9: Conn_01x04_Male, Connector_PinHeader_2.54mm:PinHeader_1x04_P2.54mm_Vertical, symbol Connector:Conn_01x04_Male
Connections:
- net +3V3: now also J9.4 (Pin_4)
- net GND: now also J9.1 (Pin_1)
- net RX: now also J9.2 (Pin_2)
- net TX: now also J9.3 (Pin_3)
Changed lines of the file:
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@@
     (stroke (width 0) (type default) (color 0 0 0 0))
   )
-  (wire (pts (xy 113.03 26.67) (xy 116.84 26.67))
+  (wire (pts (xy 115.57 26.67) (xy 119.38 26.67))
     (stroke (width 0) (type default) (color 0 0 0 0))
   )
@@
     (stroke (width 0) (type default) (color 0 0 0 0))
   )
-  (wire (pts (xy 113.03 36.83) (xy 116.84 36.83))
+  (wire (pts (xy 115.57 31.75) (xy 119.38 31.75))
     (stroke (width 0) (type default) (color 0 0 0 0))
   )
@@
     (stroke (width 0) (type default) (color 0 0 0 0))
   )
-  (wire (pts (xy 113.03 21.59) (xy 116.84 21.59))
+  (wire (pts (xy 115.57 24.13) (xy 119.38 24.13))
     (stroke (width 0) (type default) (color 0 0 0 0))
   )
@@
     (stroke (width 0) (type default) (color 0 0 0 0))
   )
-  (wire (pts (xy 113.03 31.75) (xy 116.84 31.75))
+  (wire (pts (xy 115.57 29.21) (xy 119.38 29.21))
     (stroke (width 0) (type default) (color 0 0 0 0))
   )
@@
     )
   )
-  (global_label "RX" (shape input) (at 113.03 31.75 180) (fields_autoplaced)
+  (global_label "RX" (shape input) (at 115.57 29.21 180) (fields_autoplaced)
     (effects (font (size 1.27 1.27)) (justify right))
-    (property "Intersheet References" "${INTERSHEET_REFS}" (id 0) (at 108.1374 31.6706 0)
+    (property "Intersheet References" "${INTERSHEET_REFS}" (id 0) (at 110.6774 29.1306 0)
       (effects (font (size 1.27 1.27)) (justify right) hide)
     )
@@
     )
   )
-  (global_label "TX" (shape input) (at 113.03 26.67 180) (fields_autoplaced)
+  (global_label "TX" (shape input) (at 115.57 26.67 180) (fields_autoplaced)
     (effects (font (size 1.27 1.27)) (justify right))
-    (property "Intersheet References" "${INTERSHEET_REFS}" (id 0) (at 108.4398 26.5906 0)
+    (property "Intersheet References" "${INTERSHEET_REFS}" (id 0) (at 110.9798 26.5906 0)
       (effects (font (size 1.27 1.27)) (justify right) hide)
     )
@@
     (pin "1")
   )
-  (symbol (lib_id "power:GND") (at 113.03 36.83 270) (unit 1)
+  (symbol (lib_id "power:GND") (at 115.57 31.75 270) (unit 1)
     (in_bom yes) (on_board yes)
-    (property "Reference" "#PWR0146" (id 0) (at 106.68 36.83 0)
+    (property "Reference" "#PWR0146" (id 0) (at 109.22 31.75 0)
       (effects (font (size 1.27 1.27)) hide)
     )
-    (property "Value" "GND" (id 1) (at 107.95 36.83 90))
-    (property "Footprint" "" (id 2) (at 113.03 36.83 0)
+    (property "Value" "GND" (id 1) (at 110.49 31.75 90))
+    (property "Footprint" "" (id 2) (at 115.57 31.75 0)
       (effects (font (size 1.27 1.27)) hide)
     )
-    (property "Datasheet" "" (id 3) (at 113.03 36.83 0)
+    (property "Datasheet" "" (id 3) (at 115.57 31.75 0)
       (effects (font (size 1.27 1.27)) hide)
     )
@@
     (pin "1")
   )
-  (symbol (lib_id "power:+3.3V") (at 113.03 21.59 90) (unit 1)
+  (symbol (lib_id "power:+3.3V") (at 115.57 24.13 90) (unit 1)
     (in_bom yes) (on_board yes)
-    (property "Reference" "#PWR0145" (id 0) (at 116.84 21.59 0)
+    (property "Reference" "#PWR0145" (id 0) (at 119.38 24.13 0)
       (effects (font (size 1.27 1.27)) hide)
     )
-    (property "Value" "+3.3V" (id 1) (at 107.95 21.59 90))
-    (property "Footprint" "" (id 2) (at 113.03 21.59 0)
+    (property "Value" "+3.3V" (id 1) (at 110.49 24.13 90))
+    (property "Footprint" "" (id 2) (at 115.57 24.13 0)
       (effects (font (size 1.27 1.27)) hide)
     )
-    (property "Datasheet" "" (id 3) (at 113.03 21.59 0)
+    (property "Datasheet" "" (id 3) (at 115.57 24.13 0)
       (effects (font (size 1.27 1.27)) hide)
     )
@@
     (pin "1")
   )
-  (symbol (lib_id "Connector:TestPoint") (at 116.84 21.59 270) (unit 1)
-    (in_bom yes) (on_board yes)
-    (property "Reference" "TP1" (id 0) (at 121.92 20.32 90)
-      (effects (font (size 1.27 1.27)) (justify left))
-    )
-    (property "Value" "+3.3V" (id 1) (at 121.92 22.3521 90)
-      (effects (font (size 1.27 1.27)) (justify left))
-    )
-    (property "Footprint" "TestPoint:TestPoint_Pad_D1.5mm" (id 2) (at 116.84 26.67 0)
-      (effects (font (size 1.27 1.27)) hide)
-    )
-    (property "Datasheet" "~" (id 3) (at 116.84 26.67 0)
-      (effects (font (size 1.27 1.27)) hide)
-    )
-    (pin "1")
-  )
   (symbol (lib_id "Regulator_Linear:AMS1117CD-3.3") (at 129.54 121.92 0) (unit 1)
     (in_bom yes) (on_board yes) (fields_autoplaced)
@@
     (pin "1")
   )
-  (symbol (lib_id "Connector:TestPoint") (at 116.84 31.75 270) (unit 1)
-    (in_bom yes) (on_board yes)
-    (property "Reference" "TP3" (id 0) (at 121.92 30.48 90)
-      (effects (font (size 1.27 1.27)) (justify left))
-    )
-    (property "Value" "RX" (id 1) (at 121.92 32.5121 90)
-      (effects (font (size 1.27 1.27)) (justify left))
-    )
-    (property "Footprint" "TestPoint:TestPoint_Pad_D1.5mm" (id 2) (at 116.84 36.83 0)
-      (effects (font (size 1.27 1.27)) hide)
-    )
-    (property "Datasheet" "~" (id 3) (at 116.84 36.83 0)
-      (effects (font (size 1.27 1.27)) hide)
-    )
-    (pin "1")
-  )
   (symbol (lib_id "power:GND") (at 251.46 138.43 270) (unit 1)
     (in_bom yes) (on_board yes) (fields_autoplaced)
@@
     (pin "3")
   )
-  (symbol (lib_id "Connector:TestPoint") (at 116.84 26.67 270) (unit 1)
-    (in_bom yes) (on_board yes)
-    (property "Reference" "TP2" (id 0) (at 121.92 25.4 90)
-      (effects (font (size 1.27 1.27)) (justify left))
-    )
-    (property "Value" "TX" (id 1) (at 121.92 27.4321 90)
-      (effects (font (size 1.27 1.27)) (justify left))
-    )
-    (property "Footprint" "TestPoint:TestPoint_Pad_D1.5mm" (id 2) (at 116.84 31.75 0)
-      (effects (font (size 1.27 1.27)) hide)
-    )
-    (property "Datasheet" "~" (id 3) (at 116.84 31.75 0)
-      (effects (font (size 1.27 1.27)) hide)
-    )
-    (pin "1")
-  )
   (symbol (lib_id "Device:C") (at 231.14 22.86 90) (unit 1)
     (in_bom yes) (on_board yes)
@@
     (pin "1")
   )
-  (symbol (lib_id "Connector:TestPoint") (at 116.84 36.83 270) (unit 1)
-    (in_bom yes) (on_board yes)
-    (property "Reference" "TP4" (id 0) (at 121.92 35.56 90)
-      (effects (font (size 1.27 1.27)) (justify left))
-    )
-    (property "Value" "GND" (id 1) (at 121.92 37.5921 90)
-      (effects (font (size 1.27 1.27)) (justify left))
-    )
-    (property "Footprint" "TestPoint:TestPoint_Pad_D1.5mm" (id 2) (at 116.84 41.91 0)
-      (effects (font (size 1.27 1.27)) hide)
-    )
-    (property "Datasheet" "~" (id 3) (at 116.84 41.91 0)
-      (effects (font (size 1.27 1.27)) hide)
-    )
-    (pin "1")
-  )
   (symbol (lib_id "Device:R") (at 270.51 63.5 180) (unit 1)
     (in_bom yes) (on_board yes)
@@
     (pin "2")
   )
+  (symbol (lib_id "Connector:Conn_01x04_Male") (at 124.46 29.21 180) (unit 1)
+    (in_bom yes) (on_board yes)
+    (property "Reference" "J9" (id 0) (at 121.92 33.02 0)
+      (effects (font (size 1.27 1.27)) (justify right))
+    )
+    (property "Value" "Conn_01x04_Male" (id 1) (at 125.73 35.56 90)
+      (effects (font (size 1.27 1.27)) (justify right))
+    )
+    (property "Footprint" "Connector_PinHeader_2.54mm:PinHeader_1x04_P2.54mm_Vertical" (id 2) (at 124.46 29.21 0)
+      (effects (font (size 1.27 1.27)) hide)
+    )
+    (property "Datasheet" "~" (id 3) (at 124.46 29.21 0)
+      (effects (font (size 1.27 1.27)) hide)
+    )
+    (pin "1")
+    (pin "2")
+    (pin "3")
+    (pin "4")
+  )
   (symbol (lib_id "Device:R") (at 55.88 87.63 180) (unit 1)
     (in_bom yes) (on_board yes)
@@
       (reference "J8") (unit 1) (value "Molex Micro-fit 3x1") (footprint "Connector_Molex:Molex_Micro-Fit_3.0_43650-0300_1x03_P3.00mm_Horizontal")
     )
+    (path "/f901e912-c299-49a9-b1d9-f9b63f35df46"
+      (reference "J9") (unit 1) (value "Conn_01x04_Male") (footprint "Connector_PinHeader_2.54mm:PinHeader_1x04_P2.54mm_Vertical")
+    )
     (path "/f14a0100-bc3e-4b3a-b1ca-db976ded308e"
       (reference "JP1") (unit 1) (value "SolderJumper_2_Open") (footprint "Jumper:SolderJumper-2_P1.3mm_Open_RoundedPad1.0x1.5mm")
@@
       (reference "R19") (unit 1) (value "1M") (footprint "Resistor_SMD:R_0805_2012Metric")
     )
-    (path "/63405878-cf3b-44a2-abdf-7ac907f9453d"
-      (reference "TP1") (unit 1) (value "+3.3V") (footprint "TestPoint:TestPoint_Pad_D1.5mm")
-    )
-    (path "/ab4c9366-637c-43ce-8605-21e0d4b4a7a7"
-      (reference "TP2") (unit 1) (value "TX") (footprint "TestPoint:TestPoint_Pad_D1.5mm")
-    )
-    (path "/9af74590-7b7f-4864-b1de-2868af720204"
-      (reference "TP3") (unit 1) (value "RX") (footprint "TestPoint:TestPoint_Pad_D1.5mm")
-    )
-    (path "/e0cbf46e-8228-4b92-be43-92541b68ac5e"
-      (reference "TP4") (unit 1) (value "GND") (footprint "TestPoint:TestPoint_Pad_D1.5mm")
-    )
     (path "/6f61acf9-283e-43c1-b11a-174e497e5b25"

Commit message: V2 in production
Parts:
- C1, C2: LCSC (none) -> C13585
- C10, C5, C6, C7, C8, C9: LCSC (none) -> C14663
- C11: LCSC (none) -> C1785
- C12, C4: LCSC (none) -> C1525
- C13, C14: LCSC (none) -> C96123
- C15: LCSC (none) -> C1710
- D1: LCSC (none) -> C64982
- L1: LCSC (none) -> C408449
- Q1, Q2: LCSC (none) -> C15127
- R11: LCSC (none) -> C23162
- R18, R5: LCSC (none) -> C25804
- R2: LCSC (none) -> C17801
- R3: LCSC (none) -> C21189
- R4: LCSC (none) -> C23221
- R6: LCSC (none) -> C22975
- R7, R8, R9: LCSC (none) -> C23025
- U1: LCSC (none) -> C82891
- U2: LCSC (none) -> C9865
- U6: LCSC (none) -> C168807
Changed lines of the file:
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@@
+      (effects (font (size 1.27 1.27)) hide)
+    )
+    (property "LCSC" "C13585" (id 4) (at 35.56 157.48 0)
       (effects (font (size 1.27 1.27)) hide)
     )
@@
       (effects (font (size 1.27 1.27)) hide)
     )
+    (property "LCSC" "C14663" (id 4) (at 86.36 88.9 0)
+      (effects (font (size 1.27 1.27)) hide)
+    )
     (pin "1")
     (pin "2")
@@
     (property "Datasheet" "http://www.aosmd.com/pdfs/datasheet/AO3401A.pdf" (id 3) (at 129.54 88.9 0)
       (effects (font (size 1.27 1.27)) (justify left) hide)
+    )
+    (property "LCSC" "C15127" (id 4) (at 129.54 88.9 0)
+      (effects (font (size 1.27 1.27)) hide)
     )
     (pin "1")
@@
       (effects (font (size 1.27 1.27)) hide)
     )
+    (property "LCSC" "C408449" (id 4) (at 121.92 168.91 0)
+      (effects (font (size 1.27 1.27)) hide)
+    )
     (pin "1")
     (pin "2")
@@
       (effects (font (size 1.27 1.27)) hide)
     )
+    (property "LCSC" "C14663" (id 4) (at 246.38 73.66 0)
+      (effects (font (size 1.27 1.27)) hide)
+    )
     (pin "1")
     (pin "2")
@@
     )
     (property "Datasheet" "~" (id 3) (at 43.18 157.48 0)
+      (effects (font (size 1.27 1.27)) hide)
+    )
+    (property "LCSC" "C13585" (id 4) (at 43.18 157.48 0)
       (effects (font (size 1.27 1.27)) hide)
     )
@@
       (effects (font (size 1.27 1.27)) hide)
     )
+    (property "LCSC" "C14663" (id 4) (at 231.14 73.66 0)
+      (effects (font (size 1.27 1.27)) hide)
+    )
     (pin "1")
     (pin "2")
@@
     )
     (property "Datasheet" "~" (id 3) (at 156.21 172.72 0)
+      (effects (font (size 1.27 1.27)) hide)
+    )
+    (property "LCSC" "C96123" (id 4) (at 156.21 172.72 0)
       (effects (font (size 1.27 1.27)) hide)
     )
@@
     )
     (property "Datasheet" "~" (id 3) (at 133.35 172.72 0)
+      (effects (font (size 1.27 1.27)) hide)
+    )
+    (property "LCSC" "C25804" (id 4) (at 133.35 172.72 0)
       (effects (font (size 1.27 1.27)) hide)
     )
@@
     (property "MANUFACTURER" "Texas Instruments" (id 7) (at 78.74 166.37 0)
       (effects (font (size 1.27 1.27)) (justify left bottom) hide)
+    )
+    (property "LCSC" "C9865" (id 8) (at 78.74 166.37 0)
+      (effects (font (size 1.27 1.27)) hide)
     )
     (pin "1")
@@
       (effects (font (size 1.27 1.27)) hide)
     )
+    (property "LCSC" "C1525" (id 4) (at 128.27 158.75 0)
+      (effects (font (size 1.27 1.27)) hide)
+    )
     (pin "1")
     (pin "2")
@@
       (effects (font (size 1.27 1.27)) hide)
     )
+    (property "LCSC" "C96123" (id 4) (at 148.59 172.72 0)
+      (effects (font (size 1.27 1.27)) hide)
+    )
     (pin "1")
     (pin "2")
@@
       (effects (font (size 1.27 1.27)) hide)
     )
+    (property "LCSC" "C14663" (id 4) (at 142.24 125.73 0)
+      (effects (font (size 1.27 1.27)) hide)
+    )
     (pin "1")
     (pin "2")
@@
       (effects (font (size 1.27 1.27)) hide)
     )
+    (property "LCSC" "C23221" (id 4) (at 115.57 158.75 0)
+      (effects (font (size 1.27 1.27)) hide)
+    )
     (pin "1")
     (pin "2")
@@
     )
     (property "Datasheet" "http://www.jameco.com/Jameco/Products/ProdDS/1538777.pdf" (id 3) (at 113.03 179.07 0)
+      (effects (font (size 1.27 1.27)) hide)
+    )
+    (property "LCSC" "C64982" (id 4) (at 113.03 179.07 0)
       (effects (font (size 1.27 1.27)) hide)
     )
@@
       (effects (font (size 1.27 1.27)) hide)
     )
+    (property "LCSC" "C23025" (id 4) (at 255.27 40.64 0)
+      (effects (font (size 1.27 1.27)) hide)
+    )
     (pin "1")
     (pin "2")
@@
       (effects (font (size 1.27 1.27)) hide)
     )
+    (property "LCSC" "C14663" (id 4) (at 246.38 22.86 0)
+      (effects (font (size 1.27 1.27)) hide)
+    )
     (pin "1")
     (pin "2")
@@
       (effects (font (size 1.27 1.27)) hide)
     )
+    (property "LCSC" "C23162" (id 4) (at 21.59 46.99 0)
+      (effects (font (size 1.27 1.27)) hide)
+    )
     (pin "1")
     (pin "2")
@@
       (effects (font (size 1.27 1.27)) hide)
     )
+    (property "LCSC" "C168807" (id 4) (at 129.54 121.92 0)
+      (effects (font (size 1.27 1.27)) hide)
+    )
     (pin "1")
     (pin "2")
@@
     )
     (property "Datasheet" "http://wiki.ai-thinker.com/_media/esp8266/esp8266_series_modules_user_manual_v1.1.pdf" (id 3) (at 41.91 45.72 0)
+      (effects (font (size 1.27 1.27)) hide)
+    )
+    (property "LCSC" "C82891" (id 4) (at 50.8 48.26 0)
       (effects (font (size 1.27 1.27)) hide)
     )
@@
       (effects (font (size 1.27 1.27)) hide)
     )
+    (property "LCSC" "C21189" (id 4) (at 55.88 158.75 0)
+      (effects (font (size 1.27 1.27)) hide)
+    )
     (pin "1")
     (pin "2")
@@
     )
     (property "Datasheet" "~" (id 3) (at 21.59 39.37 0)
+      (effects (font (size 1.27 1.27)) hide)
+    )
+    (property "LCSC" "C17801" (id 4) (at 21.59 39.37 0)
       (effects (font (size 1.27 1.27)) hide)
     )
@@
       (effects (font (size 1.27 1.27)) hide)
     )
+    (property "LCSC" "C23025" (id 4) (at 255.27 91.44 0)
+      (effects (font (size 1.27 1.27)) hide)
+    )
     (pin "1")
     (pin "2")
@@
       (effects (font (size 1.27 1.27)) (justify left) hide)
     )
+    (property "LCSC" "C15127" (id 4) (at 177.8 88.9 0)
+      (effects (font (size 1.27 1.27)) hide)
+    )
     (pin "1")
     (pin "2")
@@
     )
     (property "Datasheet" "~" (id 3) (at 101.6 163.83 0)
+      (effects (font (size 1.27 1.27)) hide)
+    )
+    (property "LCSC" "C1525" (id 4) (at 101.6 163.83 0)
       (effects (font (size 1.27 1.27)) hide)
     )
@@
       (effects (font (size 1.27 1.27)) hide)
     )
+    (property "LCSC" "C14663" (id 4) (at 231.14 22.86 0)
+      (effects (font (size 1.27 1.27)) hide)
+    )
     (pin "1")
     (pin "2")
@@
     )
     (property "Datasheet" "~" (id 3) (at 133.35 182.88 0)
+      (effects (font (size 1.27 1.27)) hide)
+    )
+    (property "LCSC" "C22975" (id 4) (at 133.35 182.88 0)
       (effects (font (size 1.27 1.27)) hide)
     )
@@
       (effects (font (size 1.27 1.27)) hide)
     )
+    (property "LCSC" "C1710" (id 4) (at 78.74 125.73 0)
+      (effects (font (size 1.27 1.27)) hide)
+    )
     (pin "1")
     (pin "2")
@@
       (effects (font (size 1.27 1.27)) hide)
     )
+    (property "LCSC" "C23025" (id 4) (at 255.27 35.56 0)
+      (effects (font (size 1.27 1.27)) hide)
+    )
     (pin "1")
     (pin "2")
@@
       (effects (font (size 1.27 1.27)) hide)
     )
+    (property "LCSC" "C25804" (id 4) (at 207.01 137.16 0)
+      (effects (font (size 1.27 1.27)) hide)
+    )
     (pin "1")
     (pin "2")
@@
       (effects (font (size 1.27 1.27)) hide)
     )
+    (property "LCSC" "C1785" (id 4) (at 121.92 152.4 0)
+      (effects (font (size 1.27 1.27)) hide)
+    )
